Commit message: Moved camera

File: models/urdf/car.xacro (robot description, xacro)
@@ -188,5 +188,5 @@
         <parent link="front_axle" />
         <child link="camera_link" />
-        <origin xyz="0.02 0 ${p['BOX_LZ'] + 0.02}" rpy="0 ${PI/6} 0" />
+        <origin xyz="0.2 0 ${p['BOX_LZ'] + 0.02}" rpy="0 ${PI/6} 0" />
     </joint>
     <!-- Image Frame -->
