Commit message: Add ros2_control support via 'use_ros2_control' launch argument. It provides an alternative Differential drive control to the Gazebo plugin (i.e. DiffDrive)

File: line_tracking_race_description/models/urdf/car.urdf.xacro (robot description, xacro)
@@ -6,9 +6,16 @@
             ros2 run xacro xacro -o car.urdf car.urdf.xacro
     -->
+    <xacro:arg name="use_ros2_control" default="false"/>
     <!-- ###### MODEL LINKS AND JOINTS ###### -->
     <xacro:include filename="car/car_core.xacro" />
     <!-- ###### CAMERA LINKS/JOINTS/SENSORS ###### -->
     <xacro:include filename="car/car_camera.xacro" />
-    <!-- ###### Car diff_drive plugins ###### -->
-    <xacro:include filename="car/car_diff_drive.xacro" />
+    <xacro:if value="$(arg use_ros2_control)">
+        <!-- ###### ros2_control plugins ###### -->
+        <xacro:include filename="car/car_ros2_control.xacro" />
+    </xacro:if>
+    <xacro:unless value="$(arg use_ros2_control)">
+        <!-- ###### Gazebo control plugins ###### -->
+        <xacro:include filename="car/car_gazebo_control.xacro" />
+    </xacro:unless>
 </robot>

File: line_tracking_race_description/models/urdf/car/car_core.xacro (robot description, xacro)
@@ -3,4 +3,5 @@
     <xacro:include filename="car_inertial.xacro" />
    <!-- ########### MODEL LINKS AND JOINTS ########### -->
+    <!-- Base Link -->
     <link name="chassis">
         <inertial>
@@ -74,8 +75,23 @@
     <xacro:include filename="car_wheel_macro.xacro" />
     <!-- Add wheels, only the front one are actuated -->
-    <xacro:wheel_macro name="front_left" parent="front_axle"  y="${p.BOX_LEN_Y/2}" actuated="true" props="${p}" />
-    <xacro:wheel_macro name="front_right" parent="front_axle" y="${-p.BOX_LEN_Y/2}" actuated="true" props="${p}" />
+    <xacro:wheel_macro name="front_left" parent="front_axle"  y="${p.BOX_LEN_Y/2}" props="${p}" />
+    <xacro:wheel_macro name="front_right" parent="front_axle" y="${-p.BOX_LEN_Y/2}" props="${p}" />
     <xacro:wheel_macro name="back_left" parent="chassis" x="${-p.BOX_LEN_X/2}" y="${p.BOX_LEN_Y/2}" z="${-p.BOX_LEN_Z/2}" props="${p}"/>
     <xacro:wheel_macro name="back_right" parent="chassis" x="${-p.BOX_LEN_X/2}" y="${-p.BOX_LEN_Y/2}" z="${-p.BOX_LEN_Z/2}" props="${p}"/>
+    <!--########### Gazebo plugins ###########-->
+    <gazebo>
+        <!-- <plugin filename="gz-sim-joint-state-publisher-system" name="gz::sim::systems::JointStatePublisher">
+                <topic>joint_states</topic>
+                <joint_name>axle_front_left</joint_name>
+                <joint_name>axle_front_right</joint_name>
+        </plugin> -->
+        <!-- <plugin
+            filename="gz-sim-pose-publisher-system" name="gz::sim::systems::PosePublisher">
+            <publish_link_pose>true</publish_link_pose>
+            <use_pose_vector_msg>true</use_pose_vector_msg>
+            <static_publisher>true</static_publisher>
+            <static_update_frequency>1</static_update_frequency>
+        </plugin> -->
+    </gazebo>
     <!--########### COLORS used for the links. Only in RViz, for Gazebo is different ###########-->
     <xacro:include filename="car_materials.xacro" />

File: line_tracking_race_description/models/urdf/car/car_gazebo_control.xacro (robot description, xacro)
@@ -17,19 +17,12 @@
             <max_angular_velocity>1</max_angular_velocity>
             <min_angular_velocity>-1</min_angular_velocity>
-            <odom_publish_frequency>1</odom_publish_frequency>
+            <!-- Odometry published by DiffDrive -->
+            <odom_publish_frequency>30</odom_publish_frequency>
+            <tf_topic>/tf</tf_topic>
         </plugin>
-        <plugin
-            filename="gz-sim-joint-state-publisher-system" name="gz::sim::systems::JointStatePublisher">
-        </plugin>
-        <plugin
-            filename="gz-sim-pose-publisher-system" name="gz::sim::systems::PosePublisher">
-            <publish_link_pose>true</publish_link_pose>
-            <use_pose_vector_msg>true</use_pose_vector_msg>
-            <static_publisher>true</static_publisher>
-            <static_update_frequency>1</static_update_frequency>
-        </plugin>
-        <plugin
-            filename="gz-sim-odometry-publisher-system" name="gz::sim::systems::OdometryPublisher">
-            <robot_base_frame>chassis</robot_base_frame>
+        <plugin filename="gz-sim-joint-state-publisher-system" name="gz::sim::systems::JointStatePublisher">
+                <topic>joint_states</topic>
+                <joint_name>axle_front_left</joint_name>
+                <joint_name>axle_front_right</joint_name>
         </plugin>
     </gazebo>

File: line_tracking_race_description/models/urdf/car/car_wheel_macro.xacro (robot description, xacro)
@@ -2,5 +2,5 @@
 <robot xmlns:xacro="http://www.ros.org/wiki/xacro">
     <!--########### MACRO for links and joints ###########-->
-    <xacro:macro name="wheel_macro" params="name parent x:=0 y:=0 z:=0 actuated:=false props">
+    <xacro:macro name="wheel_macro" params="name parent x:=0 y:=0 z:=0 props">
         <link name="wheel_${name}">
             <inertial>
