Commit message: Fix TF tree. Some joints were not being published.

File: line_tracking_race_description/models/urdf/car/car_core.xacro (robot description, xacro)
@@ -29,10 +29,4 @@
         <material>Gazebo/Red</material>
     </gazebo>
-    <!-- Dummy link with null inertia for KDL -->
-    <link name="dummy" />
-    <joint name="dummy_to_chassis" type="fixed">
-        <parent link="dummy" />
-        <child link="chassis" />
-    </joint>
     <!-- Frontal axle able to rotate, to which the front wheels will be connected -->
     <link name="front_axle">
@@ -79,19 +73,4 @@
     <xacro:wheel_macro name="back_left" parent="chassis" x="${-p.BOX_LEN_X/2}" y="${p.BOX_LEN_Y/2}" z="${-p.BOX_LEN_Z/2}" props="${p}"/>
     <xacro:wheel_macro name="back_right" parent="chassis" x="${-p.BOX_LEN_X/2}" y="${-p.BOX_LEN_Y/2}" z="${-p.BOX_LEN_Z/2}" props="${p}"/>
-    <!--########### Gazebo plugins ###########-->
-    <gazebo>
-        <!-- <plugin filename="gz-sim-joint-state-publisher-system" name="gz::sim::systems::JointStatePublisher">
-                <topic>joint_states</topic>
-                <joint_name>axle_front_left</joint_name>
-                <joint_name>axle_front_right</joint_name>
-        </plugin> -->
-        <!-- <plugin
-            filename="gz-sim-pose-publisher-system" name="gz::sim::systems::PosePublisher">
-            <publish_link_pose>true</publish_link_pose>
-            <use_pose_vector_msg>true</use_pose_vector_msg>
-            <static_publisher>true</static_publisher>
-            <static_update_frequency>1</static_update_frequency>
-        </plugin> -->
-    </gazebo>
     <!--########### COLORS used for the links. Only in RViz, for Gazebo is different ###########-->
     <xacro:include filename="car_materials.xacro" />

File: line_tracking_race_description/models/urdf/car/car_gazebo_control.xacro (robot description, xacro)
@@ -23,6 +23,5 @@
         <plugin filename="gz-sim-joint-state-publisher-system" name="gz::sim::systems::JointStatePublisher">
                 <topic>joint_states</topic>
-                <joint_name>axle_front_left</joint_name>
-                <joint_name>axle_front_right</joint_name>
+                <!-- publish all joints -->
         </plugin>
     </gazebo>

File: line_tracking_race_description/models/urdf/car/car_ros2_control.xacro (robot description, xacro)
@@ -26,4 +26,16 @@
             <state_interface name="position" />
         </joint>
+        <joint name="steer_front">
+            <state_interface name="position"/>
+            <state_interface name="velocity"/>
+        </joint>
+                <joint name="axle_back_left">
+            <state_interface name="position"/>
+            <state_interface name="velocity"/>
+        </joint>
+        <joint name="axle_back_right">
+            <state_interface name="position"/>
+            <state_interface name="velocity"/>
+        </joint>
         <transmission name="transmission_front_left">
             <plugin>transmission_interface/SimpleTransmission</plugin>
